Commit message: .

File: ptz_camera_description/urdf/ptz_camera1.xacro (robot description, xacro)
@@ -26,9 +26,9 @@
   <xacro:include filename="$(find ptz_camera_description)/urdf/materials.xacro" />
   <!-- Used for fixing robot to Gazebo 'base_link' -->
-  <link name="base_link"/>
+  <link name="world"/>
   <joint name="fixed" type="fixed">
-    <parent link="base_link"/>
+    <parent link="world"/>
     <child link="frame"/>
-    <origin xyz="0 0 0" rpy="0 0 0"/>
+    <origin xyz="0 0 ${frame_height/2.0}" rpy="0 0 0"/>
   </joint>
   <!-- Base Link -->
@@ -62,5 +62,5 @@
     <parent link="frame"/>
     <child link="head"/>
-    <origin xyz="0 0 ${frame_height}" rpy="0 0 0"/>
+    <origin xyz="0 ${head_height/2} 0" rpy="0 0 0"/>
     <axis xyz="0 0 1"/>
     <dynamics damping="${damping}"/>
@@ -94,5 +94,5 @@
     <parent link="head"/>
     <child link="eye"/>
-    <origin xyz="0 0 ${eye_radius+head_height}" rpy="0 0 0"/>
+    <origin xyz="0 0 ${eye_radius}" rpy="0 0 0"/>
     <axis xyz="0 1 0"/>
     <dynamics damping="${damping}"/>
@@ -100,5 +100,5 @@
   <link name="eye">
     <visual>
-    <origin xyz="0 0 0" rpy="0 0 0"/>
+    <origin xyz="0 0 ${eye_radius}" rpy="0 0 0"/>
       <geometry>
 	<sphere  radius="${eye_radius}"/>
@@ -107,5 +107,5 @@
     </visual>
     <collision>
-    <origin xyz="0 0 0" rpy="0 0 0"/>
+    <origin xyz="0 0 ${eye_radius}" rpy="0 0 0"/>
       <geometry>
 	<sphere  radius="${eye_radius}"/>
@@ -113,5 +113,5 @@
     </collision>
     <inertial>
-    <origin xyz="0 0 0" rpy="0 0 0"/>
+    <origin xyz="0 0 ${eye_radius}" rpy="0 0 0"/>
       <mass value="${mass}"/>
       <inertia
@@ -125,5 +125,5 @@
     <parent link="eye"/>
     <child link="camera"/>
-    <origin xyz="${eye_radius} 0 0 " rpy="0 0 0"/>
+    <origin xyz=" 0 ${camera_width/2} 0" rpy="0 0 0"/>
     <axis xyz="0 1 0"/>
     <dynamics damping="${damping}"/>
@@ -131,5 +131,5 @@
   <link name="camera">
     <visual>
-     <origin xyz=" 0 0 0 " rpy="0 0 0"/>
+      <origin xyz="0 0 ${camera_width/2}" rpy="0 0 0"/>
       <geometry>
 	<box size="${camera_width} ${camera_width} ${camera_width}"/>
@@ -140,5 +140,5 @@
     </visual>
     <collision>
-     <origin xyz=" 0 0 0 " rpy="0 0 0"/>
+     <origin xyz="0 0 ${camera_width/2}" rpy="0 0 0"/>
       <geometry>
 	<box size="${camera_width} ${camera_width} ${camera_width}"/>
@@ -146,5 +146,5 @@
     </collision>
     <inertial>
-     <origin xyz="0 0 0" rpy="0 0 0"/>
+     <origin xyz="0 0 ${camera_width/2}" rpy="0 0 0"/>
       <mass value="${mass}"/>
       <inertia
@@ -154,3 +154,13 @@
     </inertial>
   </link>
+  <transmission name="tran1">
+    <type>transmission_interface/SimpleTransmission</type>
+    <joint name="nec_joint">
+      <hardwareInterface>hardware_interface/EffortJointInterface</hardwareInterface>
+    </joint>
+    <actuator name="motor1">
+      <hardwareInterface>hardware_interface/EffortJointInterface</hardwareInterface>
+      <mechanicalReduction>1</mechanicalReduction>
+    </actuator>
+  </transmission>
 </robot>
